File: kicad/template.kicad_pcb (KiCad board)
At the start: 2 copper layers, 84.1 x 61.7 mm, 45 parts, among them J1 Bus_PCI_Express_x1, J4 Conn_01x04_Socket, J5 TF-115-BCP9, J6 USB_C_Receptacle_USB2.0_16P, U1 MCP25625T-E/ML, U2 RP2040, U4 W25Q128JVP, X1 ABM8-272-T3, Y1 X322516MLB4SI

Commit message: update schematic
Parts:
- moved S9 56.6 mm to (119.9, 112.8)
- moved S12 43.9 mm to (124.7, 73.8)
- moved S10 20.5 mm to (156.0, 112.0)
- moved S8 9.27 mm to (165.9, 99.3)
- moved J4 8.17 mm to (128.3, 107.4)
- moved S11 3.14 mm to (166.1, 77.5)
Connections:
- J6 pad A5: unconnected-(J6-CC1-PadA5) -> Net-(J6-CC1)
- J6 pad B5: unconnected-(J6-CC2-PadB5) -> Net-(J6-CC2)
- R11 pad 2: unconnected-(J6-CC1-PadA5) -> Net-(J6-CC1)
- R12 pad 2: unconnected-(J6-CC2-PadB5) -> Net-(J6-CC2)

Commit message: Changed Schematic
Parts:
- removed J4: Conn_01x04_Socket, Connector_Hirose:Hirose_DF13-04P-1.25DSA_1x04_P1.25mm_Vertical
- added J2: PPTC041LGBN-RC, Nicolas Library:CONN_PPTC041LGBN-RC_SUL, F.Cu at (170.9, 100.2)
- moved R10 15.5 mm to (160.8, 88.8)
- moved R9 15.5 mm to (160.8, 86.3)
- moved R8 15.5 mm to (160.8, 83.8)
- moved S8 6.03 mm to (161.5, 95.2)
- moved R7 5.02 mm to (152.8, 87.6)

Commit message: Update PCB Layout
Parts:
- added R13: 10K, Resistor_SMD:R_0603_1608Metric, F.Cu at (166.2, 104.7)
- moved J5 46.8 mm to (167.9, 86.2), turned to -90 degrees
- moved S11 40.2 mm to (128.6, 92.0)
- moved S8 40.1 mm to (123.9, 108.9)
- moved S10 21.8 mm to (134.4, 109.3)
- moved S12 19.4 mm to (118.1, 92.0)
- moved C16 16.9 mm to (172.5, 97.8)
- moved C22 16.9 mm to (172.5, 99.3)
- moved C23 16.9 mm to (172.5, 100.8)
- moved C24 16.9 mm to (172.5, 102.3)
- moved C25 16.9 mm to (172.5, 103.8)
- moved C26 16.9 mm to (172.5, 105.3)
- moved C27 16.9 mm to (172.5, 106.8)
- moved C9 16.9 mm to (172.6, 108.4)
- moved U4 15.1 mm to (156.4, 99.8), turned to 90 degrees
- moved J2 14.1 mm to (161.3, 110.5), turned to 180 degrees
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Connections:
- net /USB_D renamed /USB_N
- net CANN renamed /CANL
- net CANP renamed /CANH
- U1 pad 25: unconnected-(U1-*INT-Pad25) -> /INT
- U1 pad 29: unconnected-(U1-EPAD-Pad29) -> GND
- U2 pad 32: unconnected-(U2-GPIO21-Pad32) -> /INT
Routing:
- net /STBY: track 0.00 -> 41.9 mm, vias 0 -> 2
- net +5V: track 32.3 -> 0.00 mm, vias 2 -> 0
- net /CS_SD: track 0.00 -> 29.7 mm
- net /QSPI_SD3: track 0.00 -> 29.6 mm
- net /SCK: track 25.8 -> 53.4 mm, vias 0 -> 2
- net /QSPI_CLK: track 0.00 -> 25.6 mm
- net /RESET: track 0.00 -> 23.6 mm, vias 0 -> 2
- net /QSPI_SD0: track 0.00 -> 20.4 mm
- net /INT: track 0.00 -> 16.5 mm
- net /CS: track 0.00 -> 13.9 mm
- net /TX: track 0.00 -> 12.2 mm, vias 0 -> 2
- net /QSPI_SD2: track 0.00 -> 10.8 mm
- net /X_IN: track 2.49 -> 13.0 mm, vias 0 -> 2
- net /QSPI_SD1: track 0.00 -> 8.92 mm
- net /OSC1: track 20.3 -> 12.8 mm
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
Commit message: PCB Layout update
Parts:
- removed C1, C2: 0.1 uF, Capacitor_SMD:C_0603_1608Metric
- removed C19: 10 uF, Capacitor_SMD:C_0603_1608Metric
- removed C21, C24, C25, C26, C27: 100 nF, Capacitor_SMD:C_0603_1608Metric
- added C10: 100 nF, Capacitor_SMD:C_0402_1005Metric, F.Cu at (141.9, 105.2)
- added C11: 100 nF, Capacitor_SMD:C_0402_1005Metric, F.Cu at (139.2, 105.2)
- added C12: 100 nF, Capacitor_SMD:C_0402_1005Metric, F.Cu at (138.0, 103.4)
- added C13: 100 nF, Capacitor_SMD:C_0402_1005Metric, F.Cu at (138.0, 102.1)
- added C14: 100 nF, Capacitor_SMD:C_0402_1005Metric, F.Cu at (142.2, 100.5)
- added C15: 100 nF, Capacitor_SMD:C_0402_1005Metric, F.Cu at (141.2, 100.5)
- added C20: 100 nF, Capacitor_SMD:C_0402_1005Metric, F.Cu at (139.2, 100.5)
- added J4: Conn_01x02, Connector_PinHeader_2.54mm:PinHeader_1x02_P2.54mm_Vertical, F.Cu at (1.82, 1.82)
- C16, C18, C8, C9: footprint Capacitor_SMD:C_0603_1608Metric -> Capacitor_SMD:C_0402_1005Metric
- C17: value 15 pF -> 100 nF; footprint Capacitor_SMD:C_0603_1608Metric -> Capacitor_SMD:C_0402_1005Metric
- C22: value 100 nF -> 22 pF; footprint Capacitor_SMD:C_0603_1608Metric -> Capacitor_SMD:C_0402_1005Metric
- C23: value 100 nF -> 15 pF; footprint Capacitor_SMD:C_0603_1608Metric -> Capacitor_SMD:C_0402_1005Metric
- C3: value 0.1 uF -> 100 nF; footprint Capacitor_SMD:C_0603_1608Metric -> Capacitor_SMD:C_0402_1005Metric
- C4, C5: value 0.22 uF -> 100 nF; footprint Capacitor_SMD:C_0603_1608Metric -> Capacitor_SMD:C_0402_1005Metric
- C6: value 1 uF -> 22 pF; footprint Capacitor_SMD:C_0603_1608Metric -> Capacitor_SMD:C_0402_1005Metric
- C7: value 100 nF -> 1 uF; footprint Capacitor_SMD:C_0603_1608Metric -> Capacitor_SMD:C_0402_1005Metric
- R10, R11, R12, R13, R3, R4, R5, R6, R7, R8, R9: footprint Resistor_SMD:R_0603_1608Metric -> Resistor_SMD:R_0402_1005Metric
- moved S12 50.5 mm to (167.5, 102.7)
- moved C22 49.4 mm to (125.2, 85.1)
- moved R8 46.2 mm to (118.5, 114.4), turned to 180 degrees
- moved R7 39.2 mm to (130.0, 114.4), turned to 180 degrees
- moved R11 38.3 mm to (144.8, 112.8), turned to -90 degrees
- moved R10 37.0 mm to (118.5, 104.4), turned to 180 degrees
- moved C23 35.9 mm to (137.4, 93.5)
- moved R12 35.1 mm to (148.2, 112.8), turned to -90 degrees
- moved R13 32.8 mm to (145.9, 79.0), turned to -90 degrees
- moved C16 32.4 mm to (140.2, 100.5), turned to -90 degrees
- moved R9 29.2 mm to (130.0, 104.4), turned to 180 degrees
- moved C9 28.8 mm to (143.9, 105.2), turned to 90 degrees
- moved C6 21.4 mm to (128.8, 78.7)
- moved C17 18.4 mm to (154.5, 95.2), turned to -90 degrees
- moved C8 13.4 mm to (142.9, 105.2), turned to 90 degrees
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Connections:
- C17 pad 1: /X_IN -> GND
- C17 pad 2: GND -> +3.3V
- C22 pad 2: +3.3V -> /OSC1
- C23 pad 1: GND -> /X_IN
- C23 pad 2: +3.3V -> GND
- C4 pad 1: GND -> +3.3V
- C4 pad 2: /OSC2 -> GND
- C5 pad 1: GND -> +3.3V
- C5 pad 2: /OSC1 -> GND
- C6 pad 2: +1V1 -> /OSC2
- C7 pad 2: +1V1 -> +3.3V
- C9 pad 2: +3.3V -> +1V1
- J6 pad A4: VBUS -> unconnected-(J6-VBUS-PadA4)_1
- J6 pad A9: VBUS -> unconnected-(J6-VBUS-PadA4)
- J6 pad B4: VBUS -> unconnected-(J6-VBUS-PadA4)_2
- J6 pad B9: VBUS -> unconnected-(J6-VBUS-PadA4)_3
- R10 pad 1: /Push_B4 -> /Push_B2
- R13 pad 1: /RESET -> +3.3V
- R13 pad 2: +3.3V -> /RESET
- R8 pad 1: /Push_B2 -> /Push_B3
- R9 pad 1: /Push_B3 -> /Push_B4
- S8 pad A: unconnected-(S8-PadA) -> /Push_B2
- U2 pad 11: /Push_B1 -> unconnected-(U2-GPIO8-Pad11)
- U2 pad 24: unconnected-(U2-SWCLK-Pad24) -> /SWCLK
- U2 pad 25: unconnected-(U2-SWD-Pad25) -> /SWD
Routing:
- net +3.3V: track 16.4 -> 60.5 mm
- net /Push_B3: track 0.00 -> 40.3 mm, vias 0 -> 2
- net Net-(U2-RUN): track 0.00 -> 37.6 mm, vias 0 -> 2
- net /Push_B1: track 0.00 -> 33.1 mm, vias 0 -> 2
- net /Push_B2: track 0.00 -> 32.4 mm, vias 0 -> 2
- net /MISO: track 61.7 -> 36.3 mm, vias 3 -> 2
- net /Push_B4: track 0.00 -> 21.1 mm, vias 0 -> 2
- net /~{USB_BOOT_S}: track 0.00 -> 14.6 mm, vias 0 -> 2
- net /SCK: track 53.4 -> 39.0 mm
- net /MOSI: track 53.4 -> 41.3 mm
- net /CS_SD: track 29.7 -> 23.5 mm
- net +1V1: track 0.00 -> 5.47 mm
- net Net-(C18-Pad1): track 5.03 -> 2.59 mm
- net Net-(J6-CC1): track 0.00 -> 1.99 mm
- net Net-(J6-CC2): track 0.00 -> 1.85 mm
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
Commit message: Update PCB Layout
Parts:
- removed J4: Conn_01x02, Connector_PinHeader_2.54mm:PinHeader_1x02_P2.54mm_Vertical
- moved C3 19.8 mm to (150.9, 73.1), turned to 90 degrees
- moved C4 17.9 mm to (149.5, 79.0), turned to -90 degrees
- moved C5 16.5 mm to (147.7, 79.0), turned to -90 degrees
- moved C22 5.23 mm to (130.4, 84.7), turned to 90 degrees
- moved S12 5.13 mm to (172.6, 102.6)
- moved Y1 4.98 mm to (129.5, 81.3)
- moved C17 3.77 mm to (158.1, 94.1)
- moved U4 3.58 mm to (160.0, 99.7)
- moved C10 3.19 mm to (141.6, 108.3)
- moved C8 3.19 mm to (142.6, 108.3)
- moved C9 3.19 mm to (143.7, 108.3)
- moved R6 3.14 mm to (155.8, 102.4), turned to 180 degrees
- moved C6 0.85 mm to (128.6, 77.9), turned to -90 degrees
- moved J5 0.60 mm to (164.0, 82.9)
Routing:
- net +3.3V: track 60.5 -> 209.2 mm, vias 0 -> 7
- net /STBY: track 42.1 -> 84.8 mm, vias 2 -> 3
- net +5V: track 0.00 -> 37.9 mm, vias 0 -> 2
- net /Push_B2: track 32.4 -> 63.2 mm
- net /SDA: track 0.00 -> 30.7 mm, vias 0 -> 2
- net /SCL: track 0.00 -> 28.7 mm, vias 0 -> 2
- net +1V1: track 5.47 -> 22.4 mm, vias 0 -> 4
- net /Push_B3: track 40.3 -> 54.7 mm, vias 2 -> 4
- net /MOSI: track 41.3 -> 51.8 mm, vias 3 -> 4
- net /QSPI_SD3: track 29.6 -> 40.0 mm
- net /QSPI_SD0: track 20.4 -> 28.3 mm
- net /QSPI_CLK: track 25.6 -> 33.5 mm
- net /MISO: track 36.3 -> 44.2 mm, vias 2 -> 4
- net GND: track 0.00 -> 7.45 mm, vias 0 -> 45
- net /Push_B4: track 21.1 -> 28.2 mm, vias 2 -> 4
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- added copper zone on B.Cu, net GND
- added copper zone on F.Cu, net GND
Other:
- board text added: "Status 0.1.0"
- board text removed: "Nicolas Suarez Status Module 0.1.0"

Commit message: PCB Layout Update
Routing:
- net +BAT: track 0.00 -> 11.9 mm, vias 0 -> 1
- net +3.3V: track 209.2 -> 219.1 mm, vias 7 -> 8
- net +5V: track 37.9 -> 47.7 mm, vias 2 -> 3
- net /STBY: vias 3 -> 2
- net GND: vias 45 -> 72

Commit message: Update PCB layout
Routing:
- net /QSPI_SD3: track 40.0 -> 37.7 mm
- net /QSPI_CLK: track 33.5 -> 33.0 mm
- net GND: vias 72 -> 77
Changed lines of the file:
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@@
+	)
+	(via
+		(at 158.47 103.94)
+		(size 0.4)
+		(drill 0.3)
+		(layers "F.Cu" "B.Cu")
+		(free yes)
+		(net 17)
 	)
 	(via
@@
 	)
 	(via
+		(at 159.91 104.34)
+		(size 0.4)
+		(drill 0.3)
+		(layers "F.Cu" "B.Cu")
+		(free yes)
+		(net 17)
+	)
+	(via
 		(at 135.98 84.93)
 		(size 0.4)
@@
 	)
 	(via
+		(at 156.33 103.45)
+		(size 0.4)
+		(drill 0.3)
+		(layers "F.Cu" "B.Cu")
+		(free yes)
+		(net 17)
+	)
+	(via
 		(at 163.16 100.98)
 		(size 0.4)
@@
 	)
 	(via
+		(at 153.89 97.89)
+		(size 0.4)
+		(drill 0.3)
+		(layers "F.Cu" "B.Cu")
+		(free yes)
+		(net 17)
+	)
+	(via
 		(at 148.93 96.46)
 		(size 0.4)
@@
 	(via
 		(at 141.9352 88.4936)
+		(size 0.4)
+		(drill 0.3)
+		(layers "F.Cu" "B.Cu")
+		(free yes)
+		(net 17)
+	)
+	(via
+		(at 139.13 96.61)
 		(size 0.4)
 		(drill 0.3)
@@
 	)
 	(segment
-		(start 161.880449 96.310551)
-		(end 162.306 95.885)
-		(width 0.15)
-		(layer "F.Cu")
-		(net 39)
-	)
-	(segment
 		(start 148.53 103.433896)
 		(end 148.53 101.74)
@@
 	)
 	(segment
+		(start 161.880449 96.310551)
+		(end 162.461 95.73)
+		(width 0.15)
+		(layer "F.Cu")
+		(net 39)
+	)
+	(segment
+		(start 164.084 96.52)
+		(end 164.084 101.981)
+		(width 0.15)
+		(layer "F.Cu")
+		(net 39)
+	)
+	(segment
+		(start 150.556904 105.4608)
+		(end 148.53 103.433896)
+		(width 0.15)
+		(layer "F.Cu")
+		(net 39)
+	)
+	(segment
+		(start 160.6042 105.4608)
+		(end 150.556904 105.4608)
+		(width 0.15)
+		(layer "F.Cu")
+		(net 39)
+	)
+	(segment
 		(start 164.084 101.981)
 		(end 160.6042 105.4608)
@@
 	)
 	(segment
-		(start 160.6042 105.4608)
-		(end 150.556904 105.4608)
-		(width 0.15)
-		(layer "F.Cu")
-		(net 39)
-	)
-	(segment
-		(start 163.449 95.885)
-		(end 164.084 96.52)
-		(width 0.15)
-		(layer "F.Cu")
-		(net 39)
-	)
-	(segment
 		(start 161.880449 96.956)
 		(end 161.880449 96.310551)
@@
 	)
 	(segment
-		(start 164.084 96.52)
-		(end 164.084 101.981)
+		(start 162.461 95.73)
+		(end 163.294 95.73)
 		(width 0.15)
 		(layer "F.Cu")
@@
 	)
 	(segment
-		(start 150.556904 105.4608)
-		(end 148.53 103.433896)
+		(start 163.294 95.73)
+		(end 164.084 96.52)
 		(width 0.15)
 		(layer "F.Cu")
@@
 	)
 	(segment
-		(start 162.306 95.885)
-		(end 163.449 95.885)
-		(width 0.15)
-		(layer "F.Cu")
-		(net 39)
-	)
-	(segment
-		(start 166.497 96.393)
-		(end 166.497 103.251)
+		(start 159.340449 95.929551)
+		(end 160.5788 94.6912)
+		(width 0.15)
+		(layer "F.Cu")
+		(net 40)
+	)
+	(segment
+		(start 161.2492 106.7308)
+		(end 150.2918 106.7308)
 		(width 0.15)
 		(layer "F.Cu")
@@
 	)
 	(segment
-		(start 159.340449 95.929551)
-		(end 160.5788 94.6912)
-		(width 0.15)
-		(layer "F.Cu")
-		(net 40)
-	)
-	(segment
-		(start 164.7952 94.6912)
-		(end 166.497 96.393)
-		(width 0.15)
-		(layer "F.Cu")
-		(net 40)
-	)
-	(segment
-		(start 160.5788 94.6912)
-		(end 164.7952 94.6912)
-		(width 0.15)
-		(layer "F.Cu")
-		(net 40)
-	)
-	(segment
-		(start 163.0172 106.7308)
-		(end 150.2918 106.7308)
-		(width 0.15)
-		(layer "F.Cu")
-		(net 40)
-	)
-	(segment
 		(start 159.340449 96.956)
 		(end 159.340449 95.929551)
@@
 	)
 	(segment
-		(start 166.497 103.251)
-		(end 163.0172 106.7308)
+		(start 160.5788 94.6912)
+		(end 164.0412 94.6912)
+		(width 0.15)
+		(layer "F.Cu")
+		(net 40)
+	)
+	(segment
+		(start 164.0412 94.6912)
+		(end 165.57 96.22)
+		(width 0.15)
+		(layer "F.Cu")
+		(net 40)
+	)
+	(segment
+		(start 165.57 96.22)
+		(end 165.57 102.41)
+		(width 0.15)
+		(layer "F.Cu")
+		(net 40)
+	)
+	(segment
+		(start 165.57 102.41)
+		(end 161.2492 106.7308)
 		(width 0.15)
 		(layer "F.Cu")
@@
 	)
 	(segment
-		(start 165.227 96.774)
-		(end 163.6522 95.1992)
+		(start 163.6522 95.1992)
+		(end 161.4808 95.1992)
 		(width 0.15)
 		(layer "F.Cu")
@@
 	)
 	(segment
-		(start 161.5186 106.0704)
-		(end 165.227 102.362)
+		(start 161.4808 95.1992)
+		(end 160.610449 96.069551)
 		(width 0.15)
 		(layer "F.Cu")
@@
 	)
 	(segment
-		(start 161.8488 95.1992)
-		(end 160.610449 96.437551)
+		(start 164.78 102.15)
+		(end 164.78 96.327)
 		(width 0.15)
 		(layer "F.Cu")
@@
 	)
 	(segment
-		(start 150.4204 106.0704)
-		(end 161.5186 106.0704)
+		(start 160.610449 96.069551)
+		(end 160.610449 96.956)
 		(width 0.15)
 		(layer "F.Cu")
@@
 	)
 	(segment
-		(start 165.227 102.362)
-		(end 165.227 96.774)
+		(start 160.8596 106.0704)
+		(end 164.78 102.15)
 		(width 0.15)
 		(layer "F.Cu")
@@
 	)
 	(segment
+		(start 150.4204 106.0704)
+		(end 160.8596 106.0704)
+		(width 0.15)
+		(layer "F.Cu")
+		(net 42)
+	)
+	(segment
 		(start 148.13 103.78)
 		(end 150.4204 106.0704)
@@
 	)
 	(segment
-		(start 163.6522 95.1992)
-		(end 161.8488 95.1992)
-		(width 0.15)
-		(layer "F.Cu")
-		(net 42)
-	)
-	(segment
-		(start 160.610449 96.437551)
-		(end 160.610449 96.956)
-		(width 0.15)
-		(layer "F.Cu")
+		(start 164.78 96.327)
+		(end 163.6522 95.1992)
+		(width 0.15)
+		(layer "F.Cu")

Commit message: Update PCB Layout
Parts:
- removed S12: TS-1187A-B-A-B, Nicolas Library:SW_TS-1187A-B-A-B
- added D1: LED, LED_SMD:LED_0402_1005Metric, F.Cu at (156.1, 115.3)
- added J3: Conn_01x04, Connector:NS-Tech_Grove_1x04_P2mm_Vertical, F.Cu at (119.8, 86.8)
- added J7: Conn_01x02, Connector_PinHeader_2.54mm:PinHeader_1x02_P2.54mm_Vertical, F.Cu at (169.5, 104.2)
- added R14: 1K, Resistor_SMD:R_0402_1005Metric, F.Cu at (156.1, 117.8)
- moved R7 14.9 mm to (116.2, 108.8)
- moved S7 13.8 mm to (119.7, 112.7)
- moved S8 7.70 mm to (128.3, 107.0)
- moved S9 7.58 mm to (128.3, 118.6)
- moved R8 6.81 mm to (125.3, 114.3), turned to 90 degrees
- moved R10 6.39 mm to (124.8, 103.4)
- moved S10 6.28 mm to (136.9, 112.7)
- moved R9 5.72 mm to (133.3, 109.1)
- moved S11 2.15 mm to (118.8, 97.3)
- moved J6 0.94 mm to (146.7, 118.5)
Connections:
- net /Push_B1 renamed /Push_Left
- net /Push_B2 renamed /Push_Up
- net /Push_B3 renamed /Push_Down
- net /Push_B4 renamed /Push_Right
- S10 pad C: unconnected-(S10-PadC) -> +3.3V
- S8 pad C: unconnected-(S8-PadC) -> +3.3V
- S9 pad C: unconnected-(S9-PadC) -> (no net)
- S9 pad D: (no net) -> +3.3V
Routing:
- net +3.3V: track 219.1 -> 298.8 mm, vias 8 -> 15
- net /SWD: track 0.00 -> 45.4 mm, vias 0 -> 2
- net /SWCLK: track 0.00 -> 40.8 mm, vias 0 -> 2
- net /Push_Up: track 63.2 -> 24.5 mm
- net /Push_Down: track 54.7 -> 33.5 mm, vias 4 -> 2
- net GND: track 7.45 -> 0.00 mm, vias 77 -> 112
- net /Push_Right: track 28.2 -> 23.6 mm, vias 4 -> 2
- net +1V1: track 22.4 -> 25.9 mm, vias 4 -> 5
- net /Push_Left: track 35.2 -> 38.0 mm
- net Net-(U2-RUN): track 37.9 -> 40.3 mm
- net Net-(D1-A): track 0.00 -> 1.53 mm
- net /CS_SD: track 22.4 -> 20.9 mm
- net /SCK: track 34.6 -> 35.9 mm
- net /X_IN: track 14.5 -> 15.6 mm
- net /X_OUT: track 15.0 -> 15.9 mm
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Other:
- board text added: "+3.3V"
- board text added: "BOOT"
- board text added: "DOWN"
- board text added: "GND"
- board text added: "LEFT"
- board text added: "Reset"
- board text added: "Right"
- board text added: "SWCLK"
- board text added: "SWD"
- board text added: "UP"
