File: kicad/template.kicad_pcb (KiCad board)
At the start: 2 copper layers, 84.1 x 61.7 mm, 48 parts, among them J1 Bus_PCI_Express_x1, J2 PPTC041LGBN-RC, J3 Conn_01x04, J5 TF-115-BCP9, J6 USB_C_Receptacle_USB2.0_16P, J7 Conn_01x02, U1 MCP25625T-E/ML, U2 RP2040, U4 W25Q128JVP, X1 ABM8-272-T3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

Commit message: Update PCB Layout
Parts:
- J3: footprint Connector:NS-Tech_Grove_1x04_P2mm_Vertical -> Nicolas Library:SAMTEC_MTLW-104-X-X-S-X
- J5: value TF-115-BCP9 -> 503398-1892; footprint Nicolas Library:TF115BCP9 -> 503398-1892:MOLEX_503398-1892
- moved J5 4.33 mm to (168.0, 84.7), turned to -90 degrees
- moved J3 2.43 mm to (121.1, 84.7), turned to -90 degrees
- moved J2 0.29 mm to (161.3, 110.3)
- moved C12 0.28 mm to (138.0, 103.1)
- moved C7 0.13 mm to (140.3, 105.1)
- moved C11 0.13 mm to (139.3, 105.1)
Routing:
- net /CS_SD: track 20.9 -> 43.2 mm, vias 0 -> 2
- net /SCK: track 35.9 -> 58.2 mm, vias 2 -> 4
- net /MOSI: track 51.8 -> 69.1 mm
- net /MISO: track 43.8 -> 61.1 mm
- net /SWCLK: track 40.8 -> 37.7 mm
- net /SWD: track 45.4 -> 42.3 mm
- net GND: track 0.00 -> 1.65 mm, vias 112 -> 124
- net /RX: track 9.64 -> 9.13 mm
