File: kicad/template.kicad_sch (KiCad schematic)
At the start: 46 parts, among them J1 Bus_PCI_Express_x1, J2 PPTC041LGBN-RC, J4 Conn_01x02, J5 TF-115-BCP9, J6 USB_C_Receptacle_USB2.0_16P, U1 MCP25625T-E/ML, U2 RP2040, U4 W25Q128JVP, X1 ABM8-272-T3, Y1 X322516MLB4SI

Commit message: Update PCB Layout
Parts:
- removed J4: Conn_01x02, Connector_PinHeader_2.54mm:PinHeader_1x02_P2.54mm_Vertical, symbol Connector_Generic:Conn_01x02
- removed S12: TS-1187A-B-A-B, Nicolas Library:SW_TS-1187A-B-A-B, symbol TS-1187A-B-A-B:TS-1187A-B-A-B
- added D1: LED, LED_SMD:LED_0402_1005Metric, symbol Device:LED
- added J3: Conn_01x04, Connector:NS-Tech_Grove_1x04_P2mm_Vertical, symbol Connector_Generic:Conn_01x04
- added J7: Conn_01x02, Connector_PinHeader_2.54mm:PinHeader_1x02_P2.54mm_Vertical, symbol Connector_Generic:Conn_01x02
- added R14: 1K, Resistor_SMD:R_0402_1005Metric, symbol Device:R
Connections:
- net +3.3V: now also S10.C, S8.C, S9.C, J3.3 (Pin_3), R14.2
- net GND: now also D1.1 (K), J3.4 (Pin_4), J7.2 (Pin_2)
- net SWCLK: now also J3.1 (Pin_1)
- net SWD: now also J3.2 (Pin_2)
- net ~{USB_BOOT_S}: now also J7.1 (Pin_1)
- net Push_B1 renamed Push_Left
- net Push_B2 renamed Push_Up
- net Push_B3 renamed Push_Down
- net Push_B4 renamed Push_Right
- new net: D1.2 (A), R14.1
