File: kicad/status.kicad_pcb (KiCad board)
At the start: 4 copper layers, 84.1 x 61.7 mm, 57 parts, among them J2 PPTC041LGBN-RC, J3 Conn_01x03, J4 503398-1892, J5 Bus_PCI_Express_x1, J6 USB_C_Receptacle_USB2.0_16P, U2 RP2040, U3 MCP25625T-E/ML, U4 W25Q128JVP, X1 ABM8-272-T3, Y1 X322516MLB4SI

Commit message: PCB update
Parts:
- removed J2: PPTC041LGBN-RC, Nicolas Library:CONN_PPTC041LGBN-RC_SUL
- added U1: DM-OLED096-636, DM-OLED096-636:MODULE_DM-OLED096-636, F.Cu at (165.8, 125.9)
- moved R14 36.0 mm to (135.0, 88.7), turned to 0 degrees
- moved D1 35.6 mm to (132.5, 88.7), turned to 0 degrees
- moved C22 0.48 mm to (132.5, 82.6)
Routing:
- net /SDA: track 23.9 -> 34.1 mm
- net /SCL: track 28.2 -> 31.6 mm
- net +3.3V: track 52.4 -> 51.1 mm, vias 20 -> 19

Commit message: pcb update
Parts:
- moved R19 8.74 mm to (168.2, 75.8), turned to 0 degrees
- moved R16 8.09 mm to (176.7, 92.1)
- moved R17 4.33 mm to (174.4, 92.1), turned to 90 degrees
- moved R18 2.79 mm to (172.2, 92.1)
- moved J4 2.00 mm to (162.9, 84.1)
- moved S12 1.27 mm to (171.9, 105.0)
- moved G*** 1.15 mm to (171.0, 98.1)
Routing:
- net Net-(J4-DAT2): track 3.47 -> 11.0 mm
- net +3.3V: track 51.1 -> 56.5 mm, vias 19 -> 21
- net /MOSI: track 43.9 -> 47.4 mm
- net /CS_SD: track 35.1 -> 37.1 mm
- net Net-(J4-DAT1): track 3.43 -> 5.16 mm
- net /MISO: track 37.5 -> 38.7 mm
- net /SCK: track 30.8 -> 31.8 mm
- net /~{USB_BOOT_S}: track 19.7 -> 18.9 mm
