File: kicad/status.kicad_sch (KiCad schematic)
At the start: 56 parts, among them J3 Conn_01x03, J4 503398-1892, J5 Bus_PCI_Express_x1, J6 USB_C_Receptacle_USB2.0_16P, U1 DM-OLED096-636, U2 RP2040, U3 MCP25625T-E/ML, U4 W25Q128JVP, X1 ABM8-272-T3, Y1 X322516MLB4SI

Commit message: Organized schematic into functional blocks
Other:
- note added: "Push Buttons"
- note added: "RP2040"
- note added: "SD Card Reader"
- moved on the sheet: C10, C11, C12, C13, C14, C15, C16, C17, C20, C22, C3, C4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

Commit message: PCB layout changes
Parts:
- removed R9: 10K, Resistor_SMD:R_0402_1005Metric, symbol Device:R
- added R27: 1k, Resistor_SMD:R_0402_1005Metric, symbol Device:R
Connections:
- net +3.3V: now also R27.2
- net at S10.C: now also R27.1
Changed lines of the file:
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@@
 	(text "SD Card Reader\n"
 		(exclude_from_sim no)
-		(at 336.042 229.362 0)
+		(at 348.488 229.87 0)
 		(effects
 			(font
-				(size 1.27 1.27)
+				(size 2.54 2.54)
 			)
 		)
@@
 	(text "LCD Screen\n"
 		(exclude_from_sim no)
-		(at 254.254 256.286 0)
+		(at 258.572 255.778 0)
 		(effects
 			(font
-				(size 1.27 1.27)
+				(size 2.54 2.54)
 			)
 		)
@@
 	)
 	(symbol
-		(lib_id "Device:R")
-		(at 344.17 372.11 90)
-		(unit 1)
-		(exclude_from_sim no)
-		(in_bom yes)
-		(on_board yes)
-		(dnp no)
-		(property "Reference" "R9"
-			(at 345.44 374.65 90)
-			(effects
-				(font
-					(size 1.27 1.27)
-				)
-				(justify left)
-			)
-		)
-		(property "Value" "10K"
-			(at 345.694 369.57 90)
-			(effects
-				(font
-					(size 1.27 1.27)
-				)
-				(justify left)
-			)
-		)
-		(property "Footprint" "Resistor_SMD:R_0402_1005Metric"
-			(at 344.17 373.888 90)
-			(effects
-				(font
-					(size 1.27 1.27)
-				)
-				(hide yes)
-			)
-		)
-		(property "Datasheet" "~"
-			(at 344.17 372.11 0)
-			(effects
-				(font
-					(size 1.27 1.27)
-				)
-				(hide yes)
-			)
-		)
-		(property "Description" "Resistor"
-			(at 344.17 372.11 0)
-			(effects
-				(font
-					(size 1.27 1.27)
-				)
-				(hide yes)
-			)
-		)
-		(property "LCSC Part #" "    C60490"
-			(at 344.17 372.11 0)
-			(effects
-				(font
-					(size 1.27 1.27)
-				)
-				(hide yes)
-			)
-		)
-		(property "JLC Link" "https://jlcpcb.com/partdetail/YAGEO-RC0402FR0710KL/C60490"
-			(at 344.17 372.11 0)
-			(effects
-				(font
-					(size 1.27 1.27)
-				)
-				(hide yes)
-			)
-		)
-		(property "Arrow Part Number" ""
-			(at 344.17 372.11 0)
-			(effects
-				(font
-					(size 1.27 1.27)
-				)
-			)
-		)
-		(property "Arrow Price/Stock" ""
-			(at 344.17 372.11 0)
-			(effects
-				(font
-					(size 1.27 1.27)
-				)
-			)
-		)
-		(pin "2"
-		)
-		(pin "1"
-		)
-		(instances
-			(project "status"
-				(path "/612ece3f-e722-4b33-8111-645d24cfcf05"
-					(reference "R9")
-					(unit 1)
-				)
-			)
-		)
-	)
-	(symbol
 		(lib_id "Connector:Bus_PCI_Express_x1")
 		(at 86.36 251.46 0)
@@
 					(unit 1)
 				)
+			)
+		)
+	)
+	(symbol
+		(lib_id "Device:R")
+		(at 344.17 372.11 90)
+		(unit 1)
+		(exclude_from_sim no)
+		(in_bom yes)
+		(on_board yes)
+		(dnp no)
+		(property "Reference" "R27"
+			(at 345.44 374.65 90)
+			(effects
+				(font
+					(size 1.27 1.27)
+				)
+				(justify left)
+			)
+		)
+		(property "Value" "1k"
+			(at 345.694 369.57 90)
+			(effects
+				(font
+					(size 1.27 1.27)
+				)
+				(justify left)
+			)
+		)
+		(property "Footprint" "Resistor_SMD:R_0402_1005Metric"
+			(at 344.17 373.888 90)
+			(effects
+				(font
+					(size 1.27 1.27)
+				)
+				(hide yes)
+			)
+		)
+		(property "Datasheet" "~"
+			(at 344.17 372.11 0)
+			(effects
+				(font
+					(size 1.27 1.27)
+				)
+				(hide yes)
+			)
+		)
+		(property "Description" "Resistor"
+			(at 344.17 372.11 0)
+			(effects
+				(font
+					(size 1.27 1.27)
+				)
+				(hide yes)
+			)
+		)
+		(property "LCSC Part #" "C11702"
+			(at 344.17 372.11 0)
+			(effects
+				(font
+					(size 1.27 1.27)
+				)
+				(hide yes)
+			)
+		)
+		(property "JLC Link" "https://jlcpcb.com/partdetail/12256-0402WGF1001TCE/C11702"
+			(at 344.17 372.11 0)
+			(effects
+				(font
+					(size 1.27 1.27)
+				)
+				(hide yes)
+			)
+		)
+		(property "Arrow Part Number" ""
+			(at 344.17 372.11 0)
+			(effects
+				(font
+					(size 1.27 1.27)
+				)
+			)
+		)
+		(property "Arrow Price/Stock" ""
+			(at 344.17 372.11 0)
+			(effects
+				(font
+					(size 1.27 1.27)
+				)
+			)
+		)
+		(pin "2"
+		)
+		(pin "1"
+		)
+		(instances
+			(project "status"
+				(path "/612ece3f-e722-4b33-8111-645d24cfcf05"
+					(reference "R27")
+					(unit 1)
+				)

Commit message: Fixed DRCs
Connections:
- net at J6.A4 (VBUS), J6.A9 (VBUS): no longer J6.B4 (VBUS), J6.B9 (VBUS)
Changed lines of the file:
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@@
 		(pin "B12"
-		)
-		(pin "B4"
 		)
 		(pin "A7"
@@
 		(pin "S1"
 		)
-		(pin "B9"
-		)
 		(pin "B8"
